File: MARS_time_display/MARS_time_display.sch (KiCad schematic (older format))
At the start: 27 parts, among them Q1 2N3904, Q2 2N3904, Q3 2N3904, Q4 2N3904, U1 PIC18F27Q43, Y1 32.768KHz

Commit message: Added TTgo&Audio Schematics
Parts:
- Q1, Q2, Q3, Q4: symbol dk_Transistors-Bipolar-BJT-Single:2N3904 -> MARS_time_display-rescue:2N3904-dk_Transistors-Bipolar-BJT-Single
Connections:
- net CS renamed PIC1CS
- no-connect marks 9 -> 10
Other:
- moved on the sheet: C1, C2, C3, C4, D1, DS1, Q1, Q2, Q3, Q4, R1, R10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
